Commit message: pi is an inbuilt variable so removed mine

File: diss_ws/src/simple_eva_description/urdf/variables.xacro (robot description, xacro)
@@ -4,5 +4,5 @@
 	<xacro:property name="m_total" value="9.5"/>
 	<xacro:property name="l_total" value="0.883"/>
-	<xacro:property name="pi" value="3.1415926535"/>
+	<!--<xacro:property name="pi" value="3.1415926535"/>-->
 	<!-- Link 1 variables -->
 	<xacro:property name="l1_l" value="0.187"/>
