Commit message: Added in gazebo elements

File: diss_ws/src/simple_eva_description/urdf/simple_robot.urdf.xacro (robot description, xacro)
@@ -1,6 +1,16 @@
 <?xml version="1.0"?>
 <robot name="simple_eva" xmlns:xacro="http://www.ros.org/wiki/xacro">
+	<!-- Import variables -->
 	<xacro:include filename="$(find simple_eva_description)/urdf/variables.xacro"/>
+	<!-- Import macros -->
 	<xacro:include filename="$(find simple_eva_description)/urdf/macros.xacro"/>
+	<!-- Import gazebo elements -->
+	<xacro:include filename="$(find simple_eva_description)/urdf/simple_robot.gazebo"/>
+	<!-- Used for fixing robot to Gazebo world -->
+	<link name="world"/>
+	<joint name="fixed" type="fixed">
+		<parent link="world"/>
+		<child link="link1"/>
+	</joint>
 	<!-- 1st link -->
 	<link name="link1">
@@ -73,9 +83,3 @@
 		<xacro:box_geometry name="link6" l="${l6_l}" d="${l6_d}" w="${l6_w}" XYZ="0 0 ${l6_l/2}" RPY="0 0 0"/>
 	</link>
-	<!-- Used for fixing robot to Gazebo world -->
-	<link name="world"/>
-	<joint name="fixed" type="fixed">
-		<parent link="world"/>
-		<child link="link1"/>
-	</joint>
 </robot>
