Commit message: Added in origin to inertia and trying to fix to gazebo word

File: diss_ws/src/simple_eva_description/urdf/macros.xacro (robot description, xacro)
@@ -32,6 +32,7 @@
 	</xacro:macro>
 	<!-- Cuboid inertial macro -->
-	<xacro:macro name="box_inertial" params="m l d w">
+	<xacro:macro name="box_inertial" params="m l d w XYZ RPY">
 		<inertial>
+			<origin xyz="${XYZ}" rpy="${RPY}"/>
 			<mass value="${m}"/>
 			<inertia ixx="${(1/12)*m*((l*l) + (d*d))}"
@@ -42,6 +43,7 @@
 	</xacro:macro>
 	<!-- Cylinder inertial macro -->
-	<xacro:macro name="cylinder_inertial" params="m l r">
+	<xacro:macro name="cylinder_inertial" params="m l r XYZ RPY">
 		<inertial>
+			<origin xyz="${XYZ}" rpy="${RPY}"/>
 			<mass value="${m}"/>
 			<inertia ixx="${(1/12)*m*(3*(r*r) + (l*l))}"

File: diss_ws/src/simple_eva_description/urdf/simple_robot.urdf.xacro (robot description, xacro)
@@ -6,5 +6,5 @@
 	<link name="link1">
 		<pose>0 0 ${l1_l/2} 0 0 0</pose>
-		<xacro:box_inertial m="${m_total*(l1_l/l_total)}" l="${l1_l}" d="${l1_d}" w="${l1_w}"/>
+		<xacro:box_inertial m="${m_total*(l1_l/l_total)}" l="${l1_l}" d="${l1_d}" w="${l1_w}" XYZ="0 0 0" RPY="0 0 0"/>
 		<xacro:box_geometry name="link1" l="${l1_l}" d="${l1_d}" w="${l1_w}" XYZ="0 0 0" RPY="0 0 0"/>
 	</link>
@@ -20,5 +20,5 @@
 	<link name="link2">
 		<pose>0 0 0 0 0 0</pose>
-		<xacro:cylinder_inertial m="${m_total*(l2_l/l_total)}" l="${l2_l}" r="${l2_r}"/>
+		<xacro:cylinder_inertial m="${m_total*(l2_l/l_total)}" l="${l2_l}" r="${l2_r}" XYZ="0 0 0" RPY="0 0 0"/>
 		<xacro:cylinder_geometry name="link2" l="${l2_l}" r="${l2_r}" XYZ="0 ${l2_r} ${l2_l/2}" RPY="0 0 0"/>
 	</link>
@@ -34,5 +34,5 @@
 	<link name="link3">
 		<pose>0 0 0 0 0 0</pose>
-		<xacro:cylinder_inertial m="${m_total*(l3_l/l_total)}" l="${l3_l}" r="${l3_r}"/>
+		<xacro:cylinder_inertial m="${m_total*(l3_l/l_total)}" l="${l3_l}" r="${l3_r}" XYZ="0 0 0" RPY="0 0 0"/>
 		<xacro:cylinder_geometry name="link3" l="${l3_l}" r="${l3_r}" XYZ="0 ${-1*l3_r} ${l2_l}" RPY="0 0 0"/>
 	</link>
@@ -48,5 +48,5 @@
 	<link name="link4">
 		<pose>0 0 0 0 0 0</pose>
-		<xacro:cylinder_inertial m="${m_total*(l4_l/l_total)}" l="${l4_l}" r="${l4_r}"/>
+		<xacro:cylinder_inertial m="${m_total*(l4_l/l_total)}" l="${l4_l}" r="${l4_r}" XYZ="0 0 0" RPY="0 0 0"/>
 		<xacro:cylinder_geometry name="link4" l="${l4_l}" r="${l4_r}" XYZ="0 ${l4_r} ${l4_l/2}" RPY="0 0 0"/>
 	</link>
@@ -62,5 +62,5 @@
 	<link name="link5">
 		<pose>0 0 0 0 0 0</pose>
-		<xacro:cylinder_inertial m="${m_total*(l5_l/l_total)}" l="${l5_l}" r="${l5_r}"/>
+		<xacro:cylinder_inertial m="${m_total*(l5_l/l_total)}" l="${l5_l}" r="${l5_r}" XYZ="0 0 0" RPY="0 0 0"/>
 		<xacro:cylinder_geometry name="link5" l="${l5_l}" r="${l4_r}" XYZ="0 0 ${l5_l/2}" RPY="0 0 0"/>
 	</link>
@@ -76,6 +76,13 @@
 	<link name="link6">
 		<pose>0 0 0 0 0 0</pose>
-		<xacro:box_inertial m="${m_total*(l6_l/l_total)}" l="${l6_l}" d="${l6_d}" w="${l6_w}"/>
+		<xacro:box_inertial m="${m_total*(l6_l/l_total)}" l="${l6_l}" d="${l6_d}" w="${l6_w}" XYZ="0 0 0" RPY="0 0 0"/>
 		<xacro:box_geometry name="link6" l="${l6_l}" d="${l6_d}" w="${l6_w}" XYZ="0 0 ${l6_l/2}" RPY="0 0 0"/>
 	</link>
+	<!-- Used for fixing robot to Gazebo world -->
+	<link name="world"/>
+	<joint name="fixed" type="fixed">
+		<parent link="world"/>
+		<child link="link1"/>
+		<origin xyz="0 0 0" rpy="0 0 0"/>
+	</joint>
 </robot>

Commit message: Model is now stuck to empty world

File: diss_ws/src/simple_eva_description/urdf/macros.xacro (robot description, xacro)
@@ -32,7 +32,6 @@
 	</xacro:macro>
 	<!-- Cuboid inertial macro -->
-	<xacro:macro name="box_inertial" params="m l d w XYZ RPY">
+	<xacro:macro name="box_inertial" params="m l d w">
 		<inertial>
-			<origin xyz="${XYZ}" rpy="${RPY}"/>
 			<mass value="${m}"/>
 			<inertia ixx="${(1/12)*m*((l*l) + (d*d))}"
@@ -43,7 +42,6 @@
 	</xacro:macro>
 	<!-- Cylinder inertial macro -->
-	<xacro:macro name="cylinder_inertial" params="m l r XYZ RPY">
+	<xacro:macro name="cylinder_inertial" params="m l r">
 		<inertial>
-			<origin xyz="${XYZ}" rpy="${RPY}"/>
 			<mass value="${m}"/>
 			<inertia ixx="${(1/12)*m*(3*(r*r) + (l*l))}"
@@ -55,5 +53,5 @@
 	<!-- Joint limits macro -->
 	<xacro:macro name="joint_limits" params="upper lower">
-		<limit upper="${upper*(pi/180)}" lower="${lower*(pi/180)}" effort="30" velocity="1.0"/>
+		<limit upper="${radians(upper)}" lower="${radians(lower)}" effort="30" velocity="1.0"/>
 	</xacro:macro>
 </robot>

File: diss_ws/src/simple_eva_description/urdf/simple_robot.urdf.xacro (robot description, xacro)
@@ -5,7 +5,6 @@
 	<!-- 1st link -->
 	<link name="link1">
-		<pose>0 0 ${l1_l/2} 0 0 0</pose>
-		<xacro:box_inertial m="${m_total*(l1_l/l_total)}" l="${l1_l}" d="${l1_d}" w="${l1_w}" XYZ="0 0 0" RPY="0 0 0"/>
-		<xacro:box_geometry name="link1" l="${l1_l}" d="${l1_d}" w="${l1_w}" XYZ="0 0 0" RPY="0 0 0"/>
+		<xacro:box_inertial m="${m_total*(l1_l/l_total)}" l="${l1_l}" d="${l1_d}" w="${l1_w}"/>
+		<xacro:box_geometry name="link1" l="${l1_l}" d="${l1_d}" w="${l1_w}" XYZ="0 0 ${l1_l/2}" RPY="0 0 0"/>
 	</link>
 	<!-- 1st joint -->
@@ -15,10 +14,9 @@
 		<xacro:joint_limits upper="179" lower="-179"/>
 		<axis xyz="0 0 1"/>
-		<origin xyz="0 0 ${l1_l/2}" rpy="0 0 0"/>
+		<origin xyz="0 0 ${l1_l}" rpy="0 0 0"/>
 	</joint>
 	<!-- 2nd link -->
 	<link name="link2">
-		<pose>0 0 0 0 0 0</pose>
-		<xacro:cylinder_inertial m="${m_total*(l2_l/l_total)}" l="${l2_l}" r="${l2_r}" XYZ="0 0 0" RPY="0 0 0"/>
+		<xacro:cylinder_inertial m="${m_total*(l2_l/l_total)}" l="${l2_l}" r="${l2_r}"/>
 		<xacro:cylinder_geometry name="link2" l="${l2_l}" r="${l2_r}" XYZ="0 ${l2_r} ${l2_l/2}" RPY="0 0 0"/>
 	</link>
@@ -33,6 +31,5 @@
 	<!-- 3rd link -->
 	<link name="link3">
-		<pose>0 0 0 0 0 0</pose>
-		<xacro:cylinder_inertial m="${m_total*(l3_l/l_total)}" l="${l3_l}" r="${l3_r}" XYZ="0 0 0" RPY="0 0 0"/>
+		<xacro:cylinder_inertial m="${m_total*(l3_l/l_total)}" l="${l3_l}" r="${l3_r}"/>
 		<xacro:cylinder_geometry name="link3" l="${l3_l}" r="${l3_r}" XYZ="0 ${-1*l3_r} ${l2_l}" RPY="0 0 0"/>
 	</link>
@@ -47,6 +44,5 @@
 	<!-- 4th link -->
 	<link name="link4">
-		<pose>0 0 0 0 0 0</pose>
-		<xacro:cylinder_inertial m="${m_total*(l4_l/l_total)}" l="${l4_l}" r="${l4_r}" XYZ="0 0 0" RPY="0 0 0"/>
+		<xacro:cylinder_inertial m="${m_total*(l4_l/l_total)}" l="${l4_l}" r="${l4_r}"/>
 		<xacro:cylinder_geometry name="link4" l="${l4_l}" r="${l4_r}" XYZ="0 ${l4_r} ${l4_l/2}" RPY="0 0 0"/>
 	</link>
@@ -61,6 +57,5 @@
 	<!-- 5th link -->
 	<link name="link5">
-		<pose>0 0 0 0 0 0</pose>
-		<xacro:cylinder_inertial m="${m_total*(l5_l/l_total)}" l="${l5_l}" r="${l5_r}" XYZ="0 0 0" RPY="0 0 0"/>
+		<xacro:cylinder_inertial m="${m_total*(l5_l/l_total)}" l="${l5_l}" r="${l5_r}"/>
 		<xacro:cylinder_geometry name="link5" l="${l5_l}" r="${l4_r}" XYZ="0 0 ${l5_l/2}" RPY="0 0 0"/>
 	</link>
@@ -75,6 +70,5 @@
 	<!-- 6th link -->
 	<link name="link6">
-		<pose>0 0 0 0 0 0</pose>
-		<xacro:box_inertial m="${m_total*(l6_l/l_total)}" l="${l6_l}" d="${l6_d}" w="${l6_w}" XYZ="0 0 0" RPY="0 0 0"/>
+		<xacro:box_inertial m="${m_total*(l6_l/l_total)}" l="${l6_l}" d="${l6_d}" w="${l6_w}"/>
 		<xacro:box_geometry name="link6" l="${l6_l}" d="${l6_d}" w="${l6_w}" XYZ="0 0 ${l6_l/2}" RPY="0 0 0"/>
 	</link>
@@ -84,5 +78,4 @@
 		<parent link="world"/>
 		<child link="link1"/>
-		<origin xyz="0 0 0" rpy="0 0 0"/>
 	</joint>
 </robot>

Commit message: Added in transmission/actuator blocks into urdf

File: diss_ws/src/simple_eva_description/urdf/macros.xacro (robot description, xacro)
@@ -55,3 +55,15 @@
 		<limit upper="${radians(upper)}" lower="${radians(lower)}" effort="30" velocity="1.0"/>
 	</xacro:macro>
+	<!-- Transmission macro -->
+	<xacro:macro name="transmission_actuator" params="nameTran nameJoint nameMotor mechRed">
+		<transmission name="${nameTran}">
+			<type>transmission_interface/SimpleTransmission</type>
+			<joint name="${nameJoint}">
+				<hardwareInterface>EffortJointInterface</hardwareInterface>
+			</joint>
+			<actuator name="${nameMotor}">
+				<hardwareInterface>EffortJointInterface</hardwareInterface>
+				<mechanicalReduction>${mechRed}</mechanicalReduction>
+			</actuator>
+		</transmission>
 </robot>

File: diss_ws/src/simple_eva_description/urdf/simple_robot.urdf.xacro (robot description, xacro)
@@ -26,4 +26,6 @@
 		<origin xyz="0 0 ${l1_l}" rpy="0 0 0"/>
 	</joint>
+	<!-- 1st transmission/actuator -->
+	<xacro:transmission_actuator nameTran="tran1" nameJoint="joint1" nameMotor="motor1" mechRed="1"/>
 	<!-- 2nd link -->
 	<link name="link2">
@@ -39,4 +41,6 @@
 		<origin xyz="0 0 ${l2_l}" rpy="0 0 0"/>
 	</joint>
+	<!-- 2nd transmission/actuator -->
+	<xacro:transmission_actuator nameTran="tran2" nameJoint="joint2" nameMotor="motor2" mechRed="1"/>
 	<!-- 3rd link -->
 	<link name="link3">
@@ -52,4 +56,6 @@
 		<origin xyz="0 0 ${l3_l}" rpy="0 0 0"/>
 	</joint>
+	<!-- 3rd transmission/actuator -->
+	<xacro:transmission_actuator nameTran="tran3" nameJoint="joint3" nameMotor="motor3" mechRed="1"/>
 	<!-- 4th link -->
 	<link name="link4">
@@ -65,4 +71,6 @@
 		<origin xyz="0 0 ${l4_l}" rpy="0 0 0"/>
 	</joint>
+	<!-- 4th transmission/actuator -->
+	<xacro:transmission_actuator nameTran="tran4" nameJoint="joint4" nameMotor="motor4" mechRed="1"/>
 	<!-- 5th link -->
 	<link name="link5">
@@ -78,4 +86,6 @@
 		<origin xyz="0 0 ${l5_l}" rpy="0 0 0"/>
 	</joint>
+	<!-- 5th transmission/actuator -->
+	<xacro:transmission_actuator nameTran="tran5" nameJoint="joint5" nameMotor="motor5" mechRed="1"/>
 	<!-- 6th link -->
 	<link name="link6">
